File: brd/power-supply/power-supply.sch (KiCad schematic (older format))
At the start: 53 parts, among them J1 IEC C13, J2 PE, J3 POWER OUTPUT, J4 CONTROL, K1 RELAY_2RT, SW1 SWITCH ON, T1 2x15 100VA, U1 LM78M05CT, U2 LM1084IT-ADJ/NOPB, U3 LM1084IT-ADJ/NOPB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

Commit message: version 1.1.2-rc añadido bom y referencias mouser en esquemático, corregido fallo de máscara en pcb y generado gerber
Parts:
- removed J3: POWER OUTPUT, symbol CONN_01X07
- removed K1: RELAY_2RT, symbol RELAY_2RT
- added C20: 100nF, Capacitors_ThroughHole:C_Disc_D3_P2.5, symbol C
- added D6: RED, LEDs:LED-5MM, symbol LED-RESCUE-power-supply
- added J3: MAIN OUT, asrdi-conn:39880-0304, symbol CONN_01X04
- added J5, J6: FAN, Socket_Strips:Socket_Strip_Straight_1x03, symbol CONN_01X03
- added J7: DUAL OUT, asrdi-conn:39880-0303, symbol CONN_01X03
- added K1: RTE24005, Relays_ThroughHole:Relay_DPDT_Schrack-RT2_RM5mm, symbol RTE24xxx
- added Q1, Q2: BC547, Housings_TO-92:TO-92_Inline_Wide, symbol BC547
- added R11: 47k, Resistors_ThroughHole:Resistor_Horizontal_RM10mm, symbol R
- added R12: 47k NTC, Capacitors_ThroughHole:C_Disc_D3_P2.5, symbol RVAR
- added R13, R15: 10k, Resistors_ThroughHole:Resistor_Horizontal_RM10mm, symbol R
- added R14: 1k5, Resistors_ThroughHole:Resistor_Horizontal_RM10mm, symbol R
- added RV1, RV2: 10k, Potentiometers:Potentiometer_Bourns_3296Y_3-8Zoll_Angular_ScrewUp, symbol POT
- added U6: LM358, Housings_DIP:DIP-8__300_ELL, symbol LM358
- C1, C18, C19, C4, C5: footprint (none) -> Capacitors_ThroughHole:C_Disc_D3_P2.5; Vendor (none) -> 594-K103K15X7RF5UL2
- C10, C11, C6, C7: footprint (none) -> Capacitors_ThroughHole:C_Radial_D12.5_L25_P5; Vendor (none) -> 647-UVR1V102MHD1TO
- C12, C13, C16, C17, C2: footprint (none) -> Capacitors_ThroughHole:C_Radial_D5_L11_P2; Vendor (none) -> 140-RGA4R7M1HBK0511G
- C14, C15: footprint (none) -> Capacitors_ThroughHole:C_Disc_D3_P2.5; Vendor (none) -> 594-K104K15X7RF5UH5
- C3: footprint (none) -> Capacitors_ThroughHole:C_Radial_D16_L25_P7.5; Vendor (none) -> 647-UVZ1J102MHD
- C8, C9: footprint (none) -> Capacitors_ThroughHole:C_Radial_D5_L11_P2; Vendor (none) -> 647-UVK1H220MDD
- D1, D2: footprint (none) -> LEDs:LED-5MM; symbol LED -> LED-RESCUE-power-supply; Vendor (none) -> 696-SLX-LX5093ID
- D3: value Diode_Bridge -> BR101; footprint (none) -> asrdi-diode:BR-10; Vendor (none) -> 583-BR101
- D4: footprint (none) -> LEDs:LED-5MM; symbol LED -> LED-RESCUE-power-supply; Vendor (none) -> 696-SLX-LX5093GD
- D5: footprint (none) -> Diodes_ThroughHole:Diode_DO-41_SOD81_Horizontal_RM10; Vendor (none) -> 583-1N4007-T
- F1, F2: footprint (none) -> asrdi-fuse:Fuseholder5x20-littelfuse646; Replace (none) -> 530-5ST6.3-R; Vendor (none) -> 576-64600001223
- HS1, HS2, HS3, HS4: footprint (none) -> asrdi-heatsink:RA-T2X-xxE; Vendor (none) -> 588-RA-T2X-51E
- J1: footprint (none) -> asrdi-conn:703W-0053; Vendor (none) -> 562-703W-00/53
- J2: footprint (none) -> Divers:douille_4mm
- J4: footprint (none) -> asrdi-conn:39880-0303; Vendor (none) -> 538-39880-0303
- Q3: renamed from Q?; footprint TO-92 -> Housings_TO-92:TO-92_Inline_Wide; Vendor (none) -> 512-BC517D74Z
- R1, R2: footprint (none) -> Resistors_ThroughHole:Resistor_Horizontal_RM15mm; Vendor (none) -> 293-1.8K-RC
- R10: footprint (none) -> Resistors_ThroughHole:Resistor_Horizontal_RM10mm; Vendor (none) -> 603-CFR-25JR-52220R
- R3: footprint (none) -> Resistors_ThroughHole:Resistor_Horizontal_RM10mm; Vendor (none) -> 603-CFR-25JR-52330R
- R4: footprint (none) -> Resistors_ThroughHole:Resistor_Horizontal_RM10mm; Vendor (none) -> 603-CFR-25JR-52390R
- R5: footprint (none) -> Resistors_ThroughHole:Resistor_Horizontal_RM10mm; Vendor (none) -> 603-CFR-25JB-1K0
- R6: footprint (none) -> Resistors_ThroughHole:Resistor_Horizontal_RM10mm; Vendor (none) -> 603-CFR-25JR-523K3
- R7: footprint (none) -> Resistors_ThroughHole:Resistor_Horizontal_RM10mm; Vendor (none) -> 603-CFR-25JR-522K2
- R8, R9: footprint (none) -> Resistors_ThroughHole:Resistor_Horizontal_RM20mm; Vendor (none) -> 279-CFR200J1K0
- SW1: footprint (none) -> asrdi-switch:Carling-2M1-SP1-T2-B4-M6RE; Vendor (none) -> 691-2M1-SP1-T2B4M6RE
- T1: footprint (none) -> asrdi-trafo:VPT30-3330; Vendor (none) -> 553-VPT30-3330
- U1: footprint TO-220 -> Power_Integrations:TO-220; Vendor (none) -> 863-MC78M05CTG
- U2, U3: footprint TO-220 -> Power_Integrations:TO-220; Vendor (none) -> 511-LD1084V
- U4: footprint TO-220 -> Power_Integrations:TO-220; Vendor (none) -> 863-MC7815CTG
- U5: footprint TO-220 -> Power_Integrations:TO-220; Vendor (none) -> 863-MC7915ACTG
Connections:
- net +12V: now also J3.1 (P1)
- net +5V: now also J3.3 (P3)
- net +5VD: now also K1.A1
- net GND: now also C20.2, D6.1 (A), J3.2 (P2), J3.4 (P4), J7.2 (P2), Q1.3 (E), Q2.3 (E), R12.2, RV1.3, RV2.3, U6.4 (V-)
- net VCC: now also J7.1 (P1)
- net VEE: now also J7.3 (P3)
- net at C11.2, C13.2, C15.2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: now also K1.11
- net VCOM: now reaches C10.1, C12.1, C14.1, C3.1, C6.1, D3.3 (+), R8.1, U1.1 (IN)
- net VCOM: now also C20.1, J5.2 (P2), K1.21, R11.1, RV1.1, RV2.1, U6.8 (V+)
- net at U5.2 (IN): now also K1.14
- net at U2.3 (IN), U3.3 (IN), U4.1 (IN): now also K1.24
- net at D5.2 (A), Q3.1 (C), R10.1: now also K1.A2
- net at Q3.2 (B), R7.1: now also Q2.1 (C)
- new net: R13.2, U6.1
- new net: R11.2, R12.1, U6.2 (-), U6.6 (-)
- new net: RV1.2, U6.3 (+)
- new net: RV2.2, U6.5 (+)
- new net: R14.2, R15.2, U6.7
- new net: Q2.2 (B), R15.1
- new net: Q1.2 (B), R13.1
- new net: J6.1 (P1), Q1.1 (C)
- new net: D6.2 (K), R14.1
- new net: J5.1 (P1), J6.2 (P2)
